File: PCB files/air_flow.sch (EAGLE design)
At the start: 66 parts, among them Q1 600mA/40V, U1 LM358, U2 LM358, U3 LMV358, U4 LMV358

Commit message: updated ealge v0 to JLCPCB
Parts:
- removed Q1: 600mA/40V, SparkFun-DiscreteSemi:TRANS_NPN-P2N2222A
- removed U7: (no value), SparkFun-IC-Power:V_REG_78XXSINK
- added C11: 100uF, SparkFun-Capacitors:100UF-POLAR-RADIAL-2.5MM-25V-20%
- added J1, J2, J3, J4: (no value), SparkFun-Connectors:CONN_01
- added Q2: 200mA/40V, SparkFun-DiscreteSemi:TRANS_NPN-2N3904
- added S4, S6: STANDOFF_ELECTRICAL5-32, th_libraries:STANDOFF_ELECTRICAL5-32
- added U$26: CONN_0138MILL, th_libraries3:CONN_0138MILL
- added U5: SHTC3, SHTC3:SHTC3
Connections:
- removed net A0: MS2.GPIOA0
- removed net A3: MS2.GPIOA3
- new net N$13: MS2.GPIOTX
- new net N$14: MS2.GPIORX
- new net N$15: MS2.GPIOMISO
- new net N$16: MS2.GPIOMOSI
- new net N$17: MS2.GPIOSCK
- new net N$7: MS2.NC
- net 3.3V: now also MS2.AREF; no longer U7.OUT
- net 3V: now also C11.+, MS2.3V, U5.VDD
- net A4: now also MS2.GPIOA4
- net A5: now also MS2.GPIOA5
- net AGND: now also U$26.1; no longer U7.GND
- net D_OUT: now also MS2.GPIOA0
- net GND: now also C11.-, Q2.E, S4.P$1, S6.P$1, U5.VSS; no longer Q1.E
- net LED_ERROR: now also MS2.GPIO10
- net LED_TBD: now also MS2.GPIO9
- net N$10: now also Q2.B; no longer Q1.B
- net N$9: now also Q2.C; no longer Q1.C
- net PWM_BUZZER: now also MS2.GPIO11
- net ROTARY_A: now also MS2.GPIO6
- net ROTARY_B: now also MS2.GPIO5
- net ROTARY_SWITCH: now also MS2.GPIO13
- net SCL: now also U5.SCL
- net SDA: now also U5.SDA
- net SWITCH1: now also MS2.GPIO12
- net S_OUT: now also MS2.GPIOA3
- net VIN: no longer U7.IN
Other:
- note added: "7-bit unshifted I2C address: 0x70"
- note added: "SHTC3 Humidity 1649-1100-1-ND"
- note removed: "Not Complete need to copy pins over from above IC footprint"

Commit message: update readme
Other:
- note added: "Generic 3.3v Regulator"
- note added: "https://www.mouser.com/ProductDetail/511-LDL1117S33R"
- note removed: "Generic 3.3v Regulator https://www.digikey.com/products/en?keywords=MCP1826S-3302E%2FAB"
- note removed: "SMD equivalent: https://www.mouser.com/ProductDetail/511-LDL1117S33R"
Changed lines of the file:
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@@
 https://www.adafruit.com/category/777</text>
 <text x="-55.88" y="81.28" size="1.778" layer="91">Generic 3.3v Regulator
-https://www.digikey.com/products/en?keywords=MCP1826S-3302E%2FAB</text>
+</text>
 <text x="50.8" y="53.34" size="1.778" layer="91" align="bottom-right">Test Points</text>
 <text x="157.48" y="50.8" size="1.778" layer="91" align="bottom-right">Indicator LEDs</text>
@@
 <text x="160.02" y="40.64" size="1.778" layer="91" align="bottom-right">Error</text>
 <text x="144.78" y="40.64" size="1.778" layer="91" align="bottom-right">User Defined</text>
-<text x="-53.34" y="75.692" size="1.778" layer="91">SMD equivalent:
+<text x="-53.34" y="75.692" size="1.778" layer="91">
 https://www.mouser.com/ProductDetail/511-LDL1117S33R</text>
 <text x="241.3" y="35.56" size="1.778" layer="91" align="bottom-right">Audio Alarm
